Commit message: Refactor dummybot URDF: update inertial properties, add visual and collision elements for wheels and casters

File: module2/dummybot_description/urdf/dummybot.urdf (robot description, URDF)
Before this commit: robot dummybot, 5 links, 4 joints
Links:
- removed link back_caster
- removed link front_caster
- added link back_caster_wheel, mass 1.0; collision sphere radius=0.0499; visual sphere radius=0.0499
- added link front_caster_wheel, mass 1.0; collision sphere radius=0.0499; visual sphere radius=0.0499
Joints:
- removed joint back_caster_joint
- removed joint front_caster_joint
- removed joint wheel_left_joint
- removed joint wheel_right_joint
- added joint back_caster_wheel_joint: type fixed, parent base_link, child back_caster_wheel, origin xyz=-0.15 0.0 -0.05 rpy=0.0 1.5705 1.5705, axis 0.0 0.0 0.0
- added joint front_caster_wheel_joint: type fixed, parent base_link, child front_caster_wheel, origin xyz=0.15 0.0 -0.05 rpy=0.0 1.5705 1.5705, axis 0.0 0.0 0.0
- added joint left_wheel_joint: type continuous, parent base_link, child left_wheel, origin xyz=0.0 0.15 0.0 rpy=0.0 1.5705 1.5705, axis 0.0 0.0 1.0
- added joint right_wheel_joint: type continuous, parent base_link, child right_wheel, origin xyz=0.0 -0.15 0.0 rpy=0.0 1.5705 1.5705, axis 0.0 0.0 1.0
