Commit message: Refactor dummybot URDF: correct inertial properties and clean up visual and collision element definitions for wheels

File: module2/dummybot_description/urdf/wheels.xacro (robot description, xacro)
@@ -1,13 +1,13 @@
-<robot xmlns:xacro="http://www.ros.org/wiki/xacro" name="dummybot">
+<robot xmlns:xacro="http://www.ros.org/wiki/xacro" name="dommybot">
     <link name="left_wheel">
         <inertial>
             <origin xyz="0.0 0.0 0.0" rpy="0.0 0.0 0.0"/>
             <mass value="1.0"/>
-            <inertia ixx="1.0" ixy="0.0" ixz="0.0" iyy="1.0" iyz="0.0" izz="1.0"/>
+            <inertia ixx="0.1" ixy="0.0" ixz="0.0" iyy="0.1" iyz="0.0" izz="0.1"/>
         </inertial>
-        <visual name="left_wheel_visual">
+        <visual name="">
             <origin xyz="0.0 0.0 0.0" rpy="0.0 0.0 0.0"/>
             <geometry>
-                <cylinder radius="0.1" length="0.05"/>
+            <cylinder radius="0.1" length="0.05"/>
             </geometry>
             <material name="">
@@ -16,5 +16,5 @@
             </material>
         </visual>
-        <collision name='left_wheel_collision'>
+        <collision>
             <origin xyz="0.0 0.0 0.0" rpy="0.0 0.0 0.0"/>
             <geometry>
@@ -27,10 +27,10 @@
             <origin xyz="0.0 0.0 0.0" rpy="0.0 0.0 0.0"/>
             <mass value="1.0"/>
-            <inertia ixx="1.0" ixy="0.0" ixz="0.0" iyy="1.0" iyz="0.0" izz="1.0"/>
+            <inertia ixx="0.1" ixy="0.0" ixz="0.0" iyy="0.1" iyz="0.0" izz="0.1"/>
         </inertial>
-        <visual name="right_wheel_visual">
+        <visual name="">
             <origin xyz="0.0 0.0 0.0" rpy="0.0 0.0 0.0"/>
             <geometry>
-                <cylinder radius="0.1" length="0.05"/>
+            <cylinder radius="0.1" length="0.05"/>
             </geometry>
             <material name="">
@@ -39,5 +39,5 @@
             </material>
         </visual>
-        <collision name='right_wheel_collision'>
+        <collision>
             <origin xyz="0.0 0.0 0.0" rpy="0.0 0.0 0.0"/>
             <geometry>
