Commit message: Refactor dummybot URDF: correct inertial properties, update joint names, and improve visual element definitions

File: module2/dummybot_description/urdf/dummybot.xacro (robot description, xacro)
@@ -1,11 +1,11 @@
 <robot xmlns:xacro="http://www.ros.org/wiki/xacro" name="dummybot">
-    <xacro:include filename="$(find dummybot_description)/urdf/wheels.xacro" />
+    <xacro:include filename="$(find dummybot_description )/urdf/wheels.xacro"/>
     <link name="base_link">
         <inertial>
             <origin xyz="0.0 0.0 0.0" rpy="0.0 0.0 0.0"/>
             <mass value="1.0"/>
-            <inertia ixx="1.0" ixy="0.0" ixz="0.0" iyy="1.0" iyz="0.0" izz="1.0"/>
+            <inertia ixx="0.1" ixy="0.0" ixz="0.0" iyy="0.1" iyz="0.0" izz="0.1"/>
         </inertial>
-        <visual name="base_link_visual">
+        <visual name="">
             <origin xyz="0.0 0.0 0.0" rpy="0.0 0.0 0.0"/>
             <geometry>
@@ -24,5 +24,5 @@
         </collision>
     </link>
-    <joint name="wheel_left_joint" type="continuous">
+    <joint name="left_wheel_joint" type="continuous">
         <origin xyz="0.0 0.15 0.0" rpy="0.0 1.5705 1.5705"/>
         <parent link="base_link"/>
@@ -30,5 +30,5 @@
         <axis xyz="0.0 0.0 1.0"/>
     </joint>
-    <joint name="wheel_right_joint" type="continuous">
+    <joint name="right_wheel_joint" type="continuous">
         <origin xyz="0.0 -0.15 0.0" rpy="0.0 1.5705 1.5705"/>
         <parent link="base_link"/>
@@ -36,11 +36,11 @@
         <axis xyz="0.0 0.0 1.0"/>
     </joint>
-    <link name="front_caster">
+    <link name="front_caster_wheel">
         <inertial>
             <origin xyz="0.0 0.0 0.0" rpy="0.0 0.0 0.0"/>
             <mass value="1.0"/>
-            <inertia ixx="1.0" ixy="0.0" ixz="0.0" iyy="1.0" iyz="0.0" izz="1.0"/>
+            <inertia ixx="0.1" ixy="0.0" ixz="0.0" iyy="0.1" iyz="0.0" izz="0.1"/>
         </inertial>
-        <visual name="front_caster_visual">
+        <visual name="">
             <origin xyz="0.0 0.0 0.0" rpy="0.0 0.0 0.0"/>
             <geometry>
@@ -55,21 +55,21 @@
             <origin xyz="0.0 0.0 0.0" rpy="0.0 0.0 0.0"/>
             <geometry>
-                <sphere radius="0.0499"/>
+            <sphere radius="0.0499"/>
             </geometry>
         </collision>
     </link>
-    <joint name="front_caster_joint" type="fixed">
-        <origin xyz="0.15 0.0 -0.05" rpy="0.0 0.0 0.0"/>
+    <joint name="front_caster_wheel_joint" type="fixed">
+        <origin xyz="0.15 0.0 -0.05" rpy="0.0 1.5705 1.5705"/>
         <parent link="base_link"/>
-        <child link="front_caster"/>
+        <child link="front_caster_wheel"/>
         <axis xyz="0.0 0.0 0.0"/>
     </joint>
- <link name="back_caster">
+    <link name="back_caster_wheel">
         <inertial>
             <origin xyz="0.0 0.0 0.0" rpy="0.0 0.0 0.0"/>
             <mass value="1.0"/>
-            <inertia ixx="1.0" ixy="0.0" ixz="0.0" iyy="1.0" iyz="0.0" izz="1.0"/>
+            <inertia ixx="0.1" ixy="0.0" ixz="0.0" iyy="0.1" iyz="0.0" izz="0.1"/>
         </inertial>
-        <visual name="back_caster_visual">
+        <visual name="">
             <origin xyz="0.0 0.0 0.0" rpy="0.0 0.0 0.0"/>
             <geometry>
@@ -84,12 +84,12 @@
             <origin xyz="0.0 0.0 0.0" rpy="0.0 0.0 0.0"/>
             <geometry>
-                <sphere radius="0.0499"/>
+            <sphere radius="0.0499"/>
             </geometry>
         </collision>
     </link>
-    <joint name="back_caster_joint" type="fixed">
-        <origin xyz="-0.15 0.0 -0.05" rpy="0.0 0.0 0.0"/>
+    <joint name="back_caster_wheel_joint" type="fixed">
+        <origin xyz="-0.15 0.0 -0.05" rpy="0.0 1.5705 1.5705"/>
         <parent link="base_link"/>
-        <child link="back_caster"/>
+        <child link="back_caster_wheel"/>
         <axis xyz="0.0 0.0 0.0"/>
     </joint>

Commit message: Add lidar and camera components to dummybot model and update bridge configuration

File: module2/dummybot_description/urdf/dummybot.xacro (robot description, xacro)
@@ -1,4 +1,5 @@
 <robot xmlns:xacro="http://www.ros.org/wiki/xacro" name="dummybot">
     <xacro:include filename="$(find dummybot_description )/urdf/dummybot.gazebo"/>
+    <xacro:include filename="$(find dummybot_description )/urdf/wheels.xacro"/>
     <link name="base_link">
         <inertial>
@@ -94,3 +95,91 @@
         <axis xyz="0.0 0.0 0.0"/>
     </joint>
+    <link name="lidar_link">
+        <visual>
+            <origin xyz="0 0 0" rpy="0 0 0"/>
+            <geometry>
+                <cylinder radius="0.05" length="0.09"/>
+            </geometry>
+            <material name="lidar_material">
+                <color rgba="0 0 0 1"/>
+            </material>
+        </visual>
+        <collision>
+            <origin xyz="0 0 0" rpy="0 0 0"/>
+            <geometry>
+                <cylinder radius="0.05" length="0.09"/>
+            </geometry>
+        </collision>
+        <inertial>
+            <origin xyz="0 0 0" rpy="0 0 0"/>
+            <mass value="1"/>
+            <inertia ixx="0.3333333333333333" ixy="0" ixz="0" iyy="0.5" iyz="0" izz="0.3333333333333333"/>
+        </inertial>
+    </link>
+        <!-- Lidar Joint -->
+    <joint name="lidar_joint" type="fixed">
+        <parent link="base_link"/>
+        <child link="lidar_link"/>
+        <origin xyz="0 0 0.09" rpy="0 0 0"/>
+    </joint>
+    <!-- Camera Link -->
+    <link name="camera_link">
+        <visual>
+            <origin xyz="0 0 0" rpy="0 0 0"/>
+            <geometry>
+                <box size="0.02 0.09 0.05"/>
+            </geometry>
+            <material name="camera_material">
+                <color rgba="0.015996293361446288 0.22696587349938613 0.07036009568874305 1"/>
+            </material>
+        </visual>
+        <collision>
+            <origin xyz="0 0 0" rpy="0 0 0"/>
+            <geometry>
+                <box size="0.02 0.09 0.05"/>
+            </geometry>
+        </collision>
+        <inertial>
+            <origin xyz="0 0 0" rpy="0 0 0"/>
+            <mass value="1"/>
+            <inertia ixx="0.16666666666666666" ixy="0" ixz="0" iyy="0.16666666666666666" iyz="0" izz="0.16666666666666666"/>
+        </inertial>
+    </link>
+    <!-- Camera Joint -->
+    <joint name="camera_joint" type="fixed">
+        <parent link="base_link"/>
+        <child link="camera_link"/>
+        <origin xyz="0.23 0 0.0" rpy="0 0 0"/>
+        <axis xyz="0 1 0"/>
+        <limit lower="-1.14" upper="1.14" velocity="3.14" effort="10.0"/>
+    </joint>
+    <!-- IMU Link -->
+    <link name="imu_link">
+        <visual>
+            <origin xyz="0 0 0" rpy="0 0 0"/>
+            <geometry>
+                <box size="0.02 0.02 0.02"/>
+            </geometry>
+            <material name="camera_material">
+                <color rgba="0.015996293361446288 0.22696587349938613 0.07036009568874305 1"/>
+            </material>
+        </visual>
+        <collision>
+            <origin xyz="0 0 0" rpy="0 0 0"/>
+            <geometry>
+                <box size="0.02 0.02 0.02"/>
+            </geometry>
+        </collision>
+        <inertial>
+            <origin xyz="0 0 0" rpy="0 0 0"/>
+            <mass value="1"/>
+            <inertia ixx="0.16666666666666666" ixy="0" ixz="0" iyy="0.16666666666666666" iyz="0" izz="0.16666666666666666"/>
+        </inertial>
+    </link>
+    <!-- IMU Joint -->
+    <joint name="imu_joint" type="fixed">
+        <parent link="base_link"/>
+        <child link="imu_link"/>
+        <origin xyz="-0.1 0 0.05" rpy="0 0 0"/>
+    </joint>
 </robot>
